Commit message: add new launch file (launch_sim.launch.py) & modified description/robot_core.xacro (add base_footprint)

File: description/robot_core.xacro (robot description, xacro)
@@ -16,4 +16,13 @@
     <!-- BASE LINK -->
     <link name="base_link">
+    </link>
+    <!-- BASE FOOTPRINT JOINT-->
+    <joint name="base_footprint_joint" type="fixed">
+        <parent link="base_link"/>
+        <child link="base_footprint"/>
+        <origin xyz="0 0 0" rpy="0 0 0"/>
+    </joint>
+    <!-- BASE FOOTPRINT LINK-->
+    <link name="base_footprint">
     </link>
     <!-- CHASSIS LINK -->
