Commit message: twist mux delete

File: description/lidar.xacro (robot description, xacro)
@@ -5,5 +5,5 @@
         <parent link="chassis"/>
         <child link="laser_frame"/>
-        <origin xyz="0.122 0 0.212" rpy="0 0 0"/>
+        <origin xyz="0.122 0 0.158" rpy="0 0 0"/>
     </joint>
     <link name="laser_frame">
@@ -11,11 +11,4 @@
             <geometry>
                 <cylinder radius="0.05" length="0.04"/>
-            </geometry>
-            <material name="black"/>
-        </visual>
-        <visual>
-            <origin xyz="0 0 -0.05"/>
-            <geometry>
-                <cylinder radius="0.01" length="0.1"/>
             </geometry>
             <material name="black"/>
